File: tmc2209-breakout.kicad_pcb (KiCad board)
At the start: 2 copper layers, 31 x 36 mm, 44 parts, among them J1 Conn_01x11, J3 Conn_01x04, J4 Conn_01x02, U1 TMC2208-LA

Commit message: go
Other:
- board text added: "TMC2209"
- board text removed: "TMC2209 mk.1"
Changed lines of the file:
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@@
 		(allow_soldermask_bridges_in_footprints no)
 		(pcbplotparams
-			(layerselection 0x00010ff_ffffffff)
+			(layerselection 0x00010fc_ffffffff)
 			(plot_on_all_layers_selection 0x0000000_00000000)
 			(disableapertmacros no)
@@
 			(outputformat 1)
 			(mirror no)
-			(drillshape 0)
+			(drillshape 1)
 			(scaleselection 1)
-			(outputdirectory "Dirty Gerber/")
+			(outputdirectory "")
 		)
 	)
@@
 			(at 3.75 -3.55 90)
 			(layer "F.SilkS")
-			(hide yes)
 			(effects
 				(font
@@
 			(at 2.5 -6.26 90)
 			(layer "F.SilkS")
+			(hide yes)
 			(effects
 				(font
@@
 			(at 0 0 90)
 			(layer "F.Fab")
-			(hide yes)
 			(effects
 				(font
@@
 			)
 		)
-		(property "Footprint" "Capacitor_SMD:CP_Elec_6.3x5.4"
+		(property "Footprint" ""
 			(at 0 0 90)
 			(layer "F.Fab")
@@
 			(pintype "passive")
 		)
-		(model "${KICAD8_3DMODEL_DIR}/Capacitor_SMD.3dshapes/CP_Elec_6.3x5.4.wrl"
+		(model "${KICAD6_3DMODEL_DIR}/Capacitor_SMD.3dshapes/CP_Elec_6.3x5.4.wrl"
 			(offset
 				(xyz 0 0 0)
@@
 		(layer "Edge.Cuts")
 	)
-	(gr_text "TMC2209 mk.1\n\n"
-		(at 160.5 40.5 0)
+	(gr_text "TMC2209\n"
+		(at 160.5 40 0)
 		(layer "F.SilkS")
 		(effects
 			(font
-				(size 1 1)
-				(thickness 0.25)
-				(bold yes)
+				(size 1.5 1.5)
+				(thickness 0.3)
 			)
 		)
